File: RP2040 Base Design/RP2040 Base Design.kicad_pcb (KiCad board)
At the start: 2 copper layers, 75 x 23 mm, 28 parts, among them J1 USB_B_Micro, J2 Conn_01x02, J3 RP2040_SWD, U1 RP2040, U2 AMS1117-3.3, U3 W25Q128JVS, Y1 X322512MSB4SI

Commit message: Fixes Fix cap values #6
Parts:
- C11, C12, C13, C14, C15, C6, C9: value 1uF -> 100nF
- C8: renamed from C7; value 1uF -> 100nF
- moved C7 10.9 mm to (36.7, 29.8), turned to 0 degrees
- moved C8 10.9 mm to (25.9, 31.4), turned to 180 degrees
- moved C10 1.83 mm to (35.9, 28.1)
- moved C9 1.83 mm to (34.4, 27.1)
- renumbered C8 to C7
Changed lines of the file:
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@@
     (at 30.607 26.797 90)
     (descr "https://www.worthingtonassembly.com/perfect-0402-footprint")
-    (property "MPN - JLCPCB" "C52923")
+    (property "MPN - JLCPCB" "C1525")
     (property "Sheetfile" "RP2040.kicad_sch")
     (property "Sheetname" "RP2040")
@@
       (effects (font (size 1 1) (thickness 0.15)) (justify mirror))
     )
-    (fp_text value "1uF" (at 0 1.3 90) (layer "B.Fab") hide
+    (fp_text value "100nF" (at 0 1.3 90) (layer "B.Fab") hide
       (effects (font (size 1 1) (thickness 0.15)) (justify mirror))
     )
@@
     (at 25.908 32.385 180)
     (descr "https://www.worthingtonassembly.com/perfect-0402-footprint")
-    (property "MPN - JLCPCB" "C52923")
+    (property "MPN - JLCPCB" "C1525")
     (property "Sheetfile" "RP2040.kicad_sch")
     (property "Sheetname" "RP2040")
@@
       (effects (font (size 1 1) (thickness 0.15)) (justify mirror))
     )
-    (fp_text value "1uF" (at 0 1.3) (layer "B.Fab") hide
+    (fp_text value "100nF" (at 0 1.3) (layer "B.Fab") hide
       (effects (font (size 1 1) (thickness 0.15)) (justify mirror))
     )
@@
     (at 34.544 37.211 -90)
     (descr "https://www.worthingtonassembly.com/perfect-0402-footprint")
-    (property "MPN - JLCPCB" "C52923")
+    (property "MPN - JLCPCB" "C1525")
     (property "Sheetfile" "RP2040.kicad_sch")
     (property "Sheetname" "RP2040")
@@
       (effects (font (size 1 1) (thickness 0.15)) (justify mirror))
     )
-    (fp_text value "1uF" (at 0 1.3 90) (layer "B.Fab") hide
+    (fp_text value "100nF" (at 0 1.3 90) (layer "B.Fab") hide
       (effects (font (size 1 1) (thickness 0.15)) (justify mirror))
     )
@@
   )
   (footprint "Custom_Footprints:Perfect_0402" (layer "B.Cu")
-    (at 35.941 28.067 90)
-    (descr "https://www.worthingtonassembly.com/perfect-0402-footprint")
-    (property "MPN - JLCPCB" "C52923")
+    (at 34.417 27.051 90)
+    (descr "https://www.worthingtonassembly.com/perfect-0402-footprint")
+    (property "MPN - JLCPCB" "C1525")
     (property "Sheetfile" "RP2040.kicad_sch")
     (property "Sheetname" "RP2040")
@@
       (effects (font (size 1 1) (thickness 0.15)) (justify mirror))
     )
-    (fp_text value "1uF" (at 0 1.3 90) (layer "B.Fab") hide
+    (fp_text value "100nF" (at 0 1.3 90) (layer "B.Fab") hide
       (effects (font (size 1 1) (thickness 0.15)) (justify mirror))
     )
@@
     (at 37.084 32.512)
     (descr "https://www.worthingtonassembly.com/perfect-0402-footprint")
-    (property "MPN - JLCPCB" "C52923")
+    (property "MPN - JLCPCB" "C1525")
     (property "Sheetfile" "RP2040.kicad_sch")
     (property "Sheetname" "RP2040")
@@
       (effects (font (size 1 1) (thickness 0.15)) (justify mirror))
     )
-    (fp_text value "1uF" (at 0 1.3) (layer "B.Fab") hide
+    (fp_text value "100nF" (at 0 1.3) (layer "B.Fab") hide
       (effects (font (size 1 1) (thickness 0.15)) (justify mirror))
     )
@@
   )
   (footprint "Custom_Footprints:Perfect_0402" (layer "B.Cu")
-    (at 34.417 27.051 90)
+    (at 35.941 28.067 90)
     (descr "https://www.worthingtonassembly.com/perfect-0402-footprint")
     (property "MPN - JLCPCB" "C52923")
@@
     (at 30.6164 38.0084 -90)
     (descr "https://www.worthingtonassembly.com/perfect-0402-footprint")
-    (property "MPN - JLCPCB" "C52923")
+    (property "MPN - JLCPCB" "C1525")
     (property "Sheetfile" "RP2040.kicad_sch")
     (property "Sheetname" "RP2040")
@@
       (effects (font (size 1 1) (thickness 0.15)) (justify mirror))
     )
-    (fp_text value "1uF" (at 0 1.3 90) (layer "B.Fab") hide
+    (fp_text value "100nF" (at 0 1.3 90) (layer "B.Fab") hide
       (effects (font (size 1 1) (thickness 0.15)) (justify mirror))
     )
@@
   )
   (footprint "Custom_Footprints:Perfect_0402" (layer "B.Cu")
-    (at 25.908 31.369 180)
+    (at 36.703 29.845)
     (descr "https://www.worthingtonassembly.com/perfect-0402-footprint")
     (property "MPN - JLCPCB" "C52923")
@@
     (clearance 0.15)
     (attr smd)
-    (fp_text reference "C8" (at 0 -1.3) (layer "B.Fab") hide
+    (fp_text reference "C7" (at 0 -1.3) (layer "B.Fab") hide
       (effects (font (size 1 1) (thickness 0.15)) (justify mirror))
     )
@@
     (fp_line (start -0.5 0.3) (end 0.55 0.3) (layer "B.Fab") (width 0.1))
     (fp_line (start -0.5 -0.3) (end 0.55 -0.3) (layer "B.Fab") (width 0.1))
-    (pad "1" smd rect (at -0.5 0 180) (size 0.6 0.7) (layers "B.Cu" "B.Paste" "B.Mask")
+    (pad "1" smd rect (at -0.5 0) (size 0.6 0.7) (layers "B.Cu" "B.Paste" "B.Mask")
       (net 6 "+1V1") (pintype "passive"))
-    (pad "2" smd rect (at 0.5 0 180) (size 0.6 0.7) (layers "B.Cu" "B.Paste" "B.Mask")
+    (pad "2" smd rect (at 0.5 0) (size 0.6 0.7) (layers "B.Cu" "B.Paste" "B.Mask")
       (net 2 "GND") (pintype "passive"))
     (model "${KICAD6_3DMODEL_DIR}/Capacitor_SMD.3dshapes/C_0402_1005Metric.step"
@@
     (at 37.084 31.496)
     (descr "https://www.worthingtonassembly.com/perfect-0402-footprint")
-    (property "MPN - JLCPCB" "C52923")
+    (property "MPN - JLCPCB" "C1525")
     (property "Sheetfile" "RP2040.kicad_sch")
     (property "Sheetname" "RP2040")
@@
       (effects (font (size 1 1) (thickness 0.15)) (justify mirror))
     )
-    (fp_text value "1uF" (at 0 1.3) (layer "B.Fab") hide
+    (fp_text value "100nF" (at 0 1.3) (layer "B.Fab") hide
       (effects (font (size 1 1) (thickness 0.15)) (justify mirror))
     )
@@
   )
   (footprint "Custom_Footprints:Perfect_0402" (layer "B.Cu")
-    (at 36.703 29.845)
-    (descr "https://www.worthingtonassembly.com/perfect-0402-footprint")
-    (property "MPN - JLCPCB" "C52923")
-    (property "Sheetfile" "RP2040.kicad_sch")
-    (property "Sheetname" "RP2040")
-    (clearance 0.15)
-    (attr smd)
-    (fp_text reference "C7" (at 0 -1.3) (layer "B.Fab") hide
-      (effects (font (size 1 1) (thickness 0.15)) (justify mirror))
-    )
-    (fp_text value "1uF" (at 0 1.3) (layer "B.Fab") hide
-      (effects (font (size 1 1) (thickness 0.15)) (justify mirror))
-    )
-    (fp_line (start -0.1 -0.4) (end 0.115672 -0.4) (layer "B.SilkS") (width 0.12))
-    (fp_line (start -0.1 0.4) (end 0.115672 0.4) (layer "B.SilkS") (width 0.12))
-    (fp_line (start 1.05 -0.5) (end -1.05 -0.5) (layer "B.CrtYd") (width 0.05))
-    (fp_line (start -1.05 0.5) (end 1.05 0.5) (layer "B.CrtYd") (width 0.05))
-    (fp_line (start 1.05 0.5) (end 1.05 -0.5) (layer "B.CrtYd") (width 0.05))
-    (fp_line (start -1.05 0.5) (end -1.05 -0.5) (layer "B.CrtYd") (width 0.05))
-    (fp_line (start -0.5 -0.3) (end 0.55 -0.3) (layer "B.Fab") (width 0.1))
-    (fp_line (start -0.5 0.3) (end 0.55 0.3) (layer "B.Fab") (width 0.1))
-    (pad "1" smd rect (at -0.5 0) (size 0.6 0.7) (layers "B.Cu" "B.Paste" "B.Mask")
+    (at 25.908 31.369 180)
+    (descr "https://www.worthingtonassembly.com/perfect-0402-footprint")
+    (property "MPN - JLCPCB" "C1525")
+    (property "Sheetfile" "RP2040.kicad_sch")
+    (property "Sheetname" "RP2040")
+    (clearance 0.15)
+    (attr smd)
+    (fp_text reference "C8" (at 0 -1.3) (layer "B.Fab") hide
+      (effects (font (size 1 1) (thickness 0.15)) (justify mirror))
+    )
+    (fp_text value "100nF" (at 0 1.3) (layer "B.Fab") hide
+      (effects (font (size 1 1) (thickness 0.15)) (justify mirror))
+    )
+    (fp_line (start -0.1 -0.4) (end 0.115672 -0.4) (layer "B.SilkS") (width 0.12))
+    (fp_line (start -0.1 0.4) (end 0.115672 0.4) (layer "B.SilkS") (width 0.12))
+    (fp_line (start 1.05 -0.5) (end -1.05 -0.5) (layer "B.CrtYd") (width 0.05))
+    (fp_line (start -1.05 0.5) (end 1.05 0.5) (layer "B.CrtYd") (width 0.05))
+    (fp_line (start 1.05 0.5) (end 1.05 -0.5) (layer "B.CrtYd") (width 0.05))
+    (fp_line (start -1.05 0.5) (end -1.05 -0.5) (layer "B.CrtYd") (width 0.05))
+    (fp_line (start -0.5 -0.3) (end 0.55 -0.3) (layer "B.Fab") (width 0.1))
+    (fp_line (start -0.5 0.3) (end 0.55 0.3) (layer "B.Fab") (width 0.1))
+    (pad "1" smd rect (at -0.5 0 180) (size 0.6 0.7) (layers "B.Cu" "B.Paste" "B.Mask")
       (net 6 "+1V1") (pintype "passive"))
-    (pad "2" smd rect (at 0.5 0) (size 0.6 0.7) (layers "B.Cu" "B.Paste" "B.Mask")
+    (pad "2" smd rect (at 0.5 0 180) (size 0.6 0.7) (layers "B.Cu" "B.Paste" "B.Mask")
       (net 2 "GND") (pintype "passive"))
     (model "${KICAD6_3DMODEL_DIR}/Capacitor_SMD.3dshapes/C_0402_1005Metric.step"
